Commit message: returning to good commit

File: src/auto_mobile_robot/models/auto_mobile_robot.urdf (robot description, URDF)
Before this commit: robot auto_mobile_robot, 6 links, 5 joints
Links:
- added link camera_depth_link
- added link camera_link
Joints:
- added joint cam_joint: type fixed, parent base_link, child camera_link, origin xyz=0.34 0 0.15 rpy=0 0 0
- added joint depth_cam_joint: type fixed, parent base_link, child camera_depth_link, origin xyz=0.34 0 0.55 rpy=-1.5707 0 -1.5707
