Commit message: a step twards making ackermann robot

File: src/auto_car/urdf/car.urdf.xacro (robot description, xacro)
@@ -4,4 +4,7 @@
     <xacro:include filename="./wheel.xacro" />
     <xacro:include filename="./sensors.xacro" />
+    <xacro:include filename="./ros_interface.xacro" />
+    <xacro:property name="x_position" value="0.25"/>
+    <xacro:property name="y_position" value="0.2"/>
     <link name="base_link">
         <visual>
@@ -11,5 +14,5 @@
             </geometry>
             <material name="yellow">
-                <color rgba="1 1 0.0 1.0"/>
+                <color rgba="1 1 0.0 0.6"/>
             </material>
         </visual>
@@ -21,7 +24,82 @@
         </collision>
     </link>
-    <xacro:wheel name="wheel_fr" x="0.3" y="0.3" z="0"/>
-    <xacro:wheel name="wheel_fl" x="0.3" y="-0.3" z="0"/>
-    <xacro:wheel name="wheel_rr" x="-0.3" y="0.3" z="0"/>
-    <xacro:wheel name="wheel_rl" x="-0.3" y="-0.3" z="0"/>
+    <!-- Define steering joint -->
+    <joint name="steering_joint" type="planar">
+        <origin xyz="0.15 0 0" rpy="0 0 0" />
+        <parent link="base_link" />
+        <child link="steering_link" />
+        <!-- <axis xyz="0 0 1" /> -->
+        <!-- <limit lower="-0.5" upper="0.5" effort="10" velocity="1" /> -->
+    </joint>
+        <!-- Define steering link -->
+    <link name="steering_link">
+        <visual>
+            <origin xyz="0 0 0" rpy="0 0 0" />
+            <geometry>
+                <box size="0.01 0.2 0.01" />
+            </geometry>
+            <material name="blue">
+                <color rgba="0 0 1 0.6"/>
+            </material>
+        </visual>
+        <collision>
+            <origin xyz="0 0 0" rpy="0 0 0" />
+            <geometry>
+                <box size="0.01 0.2 0.01" />
+            </geometry>
+        </collision>
+    </link>
+    <joint name="steering_l_joint" type="revolute">
+        <origin xyz="0 +0.1 0" rpy="0 0 0" />
+        <parent link="steering_link" />
+        <child link="steering_l_link" />
+        <axis xyz="0 0 1" />
+        <limit lower="-0.5" upper="0.5" effort="10" velocity="1" />
+    </joint>
+    <link name="steering_l_link">
+        <visual>
+            <origin xyz="0.1 0 0" rpy="0 0 0" />
+            <geometry>
+                <box size="0.2 0.01 0.01" />
+            </geometry>
+            <material name="blue">
+                <color rgba="0 0 1 0.6"/>
+            </material>
+        </visual>
+        <collision>
+            <origin xyz="0.1 0 0" rpy="0 0 0" />
+            <geometry>
+                <box size="0.2 0.01 0.01" />
+            </geometry>
+        </collision>
+    </link>
+    <joint name="steering_r_joint" type="revolute">
+        <origin xyz="0 -0.1 0" rpy="0 0 0" />
+        <parent link="steering_link" />
+        <child link="steering_r_link" />
+        <axis xyz="0 0 1" />
+        <limit lower="-0.5" upper="0.5" effort="10" velocity="1" />
+    </joint>
+    <link name="steering_r_link">
+        <visual>
+            <origin xyz="0.1 0 0" rpy="0 0 0" />
+            <geometry>
+                <box size="0.2 0.01 0.01" />
+            </geometry>
+            <material name="blue">
+                <color rgba="0 0 1 0.6"/>
+            </material>
+        </visual>
+        <collision>
+            <origin xyz="0.1 0 0" rpy="0 0 0" />
+            <geometry>
+                <box size="0.2 0.01 0.01" />
+            </geometry>
+        </collision>
+    </link>
+    <!-- Define front wheel joints connected to steering link -->
+    <xacro:steering_wheel name="wheel_fr" x="0.25" y="-0.02" parent="steering_r"/>
+    <xacro:steering_wheel name="wheel_fl" x="0.25" y="+0.02" parent="steering_l"/>
+    <xacro:wheel name="wheel_br" x="-${x_position}"  y="-${y_position}"  z="0"  parent="base" />
+    <xacro:wheel name="wheel_bl" x="-${x_position}"  y="+${y_position}"  z="0"  parent="base" />
 </robot>

File: src/auto_car/urdf/sensors.xacro (robot description, xacro)
@@ -2,8 +2,10 @@
 <robot xmlns:xacro="http://ros.org/wiki/xacro">
     <!-- Define properties for reuse -->
-    <xacro:property name="imu_update_rate" value="100"/>
-    <xacro:property name="lidar_update_rate" value="100"/>
-    <xacro:property name="camera_update_rate" value="30"/>
-    <xacro:property name="depth_camera_update_rate" value="30"/>
+    <xacro:property name="imu_update_rate"            value="100"/>
+    <xacro:property name="lidar_update_rate"          value="100"/>
+    <xacro:property name="camera_update_rate"         value="30"/>
+    <xacro:property name="depth_camera_update_rate"   value="30"/>
+    <xacro:property name="camera_x_position"          value="0.25"/>
+    <xacro:property name="camera_z_position"          value="0.07"/>
     <!-- *********************** IMU SENSOR SETUP **************************  -->
     <link name="imu_link">
@@ -145,10 +147,10 @@
     <link name="camera_link">
         <visual>
-            <origin xyz="0 0 0" rpy="0 0 0" />
+            <origin xyz="-0.02 0 0" rpy="0 0 0" />
             <geometry>
                 <box size="0.03 0.05 0.03" />
             </geometry>
             <material name="red">
-                <color rgba="1 0.0 0.0 1.0"/>
+                <color rgba="1 0.0 0.0 0.6"/>
             </material>
         </visual>
@@ -195,5 +197,5 @@
         <parent link="base_link"/>
         <child link="camera_link"/>
-        <origin        xyz="0.5 0 0.2"        rpy="0 1.5707 0" />
+        <origin        xyz="${camera_x_position} 0 ${camera_z_position}"        rpy="0 1.5707 0" />
     </joint>
     <!-- *********************** DEPTH CAMERA ****************************** -->
@@ -244,5 +246,5 @@
         <parent link="base_link"/>
         <child link="camera_depth_link"/>
-        <origin        xyz="0 0 0"        rpy="0 0 0" />
+        <origin        xyz="${camera_x_position} 0 ${camera_z_position}"        rpy="0 1.5707 0" />
     </joint>
 </robot>

File: src/auto_car/urdf/wheel.xacro (robot description, xacro)
@@ -1,6 +1,5 @@
 <?xml version="1.0"?>
 <robot xmlns:xacro="http://ros.org/wiki/xacro">
-<!-- TODO: xacro macro for wheel, params name x y z  -->
-    <xacro:macro name="wheel" params="name x y z">
+    <xacro:macro name="wheel" params="name x y z parent">
         <!-- <gazebo reference="base_link">                 <kinematic>true</kinematic>                                        <selfCollide>true</selfCollide>           <material>Gazebo/Orange</material>          </gazebo> -->
         <link name="${name}_link">
@@ -11,9 +10,9 @@
                 </geometry>
                 <material name="grey">
-                    <color rgba="0.1 0.1 0.1 1.0"/>
+                    <color rgba="0.1 0.1 0.1 0.6"/>
                 </material>
             </visual>
             <collision>
-                <origin xyz="${x} ${y} ${z}" rpy="0 0 0" />
+                <origin xyz="0 0 0" rpy="0 0 0" />
                 <geometry>
                     <cylinder radius="0.1" length="0.05" />
@@ -22,9 +21,34 @@
         </link>
         <joint name="${name}_joint" type="continuous">
-            <origin xyz="${x} ${y} ${z}" rpy="1.5707 0 0" />
-            <parent link="base_link" />
+            <origin xyz="${x} ${y} ${z}" rpy="-1.5707 0 0" />
+            <parent link="${parent}_link" />
             <child link="${name}_link" />
             <axis xyz="0 0 1" />
         </joint>
     </xacro:macro>
+    <xacro:macro name="steering_wheel" params="name x y parent">
+        <joint name="${name}_joint" type="continuous">
+            <origin xyz="${x} ${y} 0" rpy="-1.5707 0 0" />
+            <parent link="${parent}_link" />
+            <child link="${name}_link" />
+            <axis xyz="0 0 1" />
+        </joint>
+        <link name="${name}_link">
+            <visual>
+                <origin xyz="0 0 0" rpy="0 0 0" />
+                <geometry>
+                    <cylinder radius="0.1" length="0.05" />
+                </geometry>
+                <material name="grey">
+                    <color rgba="0.1 0.1 0.1 0.6"/>
+                </material>
+            </visual>
+            <collision>
+                <origin xyz="0 0 0" rpy="0 0 0" />
+                <geometry>
+                    <cylinder radius="0.1" length="0.05" />
+                </geometry>
+            </collision>
+        </link>
+    </xacro:macro>
 </robot>

Commit message: shitty ignition

File: src/auto_car/urdf/car.urdf.xacro (robot description, xacro)
@@ -25,9 +25,9 @@
     </link>
     <!-- Define steering joint -->
-    <joint name="steering_joint" type="planar">
+    <joint name="steering_joint" type="continuous">
         <origin xyz="0.15 0 0" rpy="0 0 0" />
         <parent link="base_link" />
         <child link="steering_link" />
-        <!-- <axis xyz="0 0 1" /> -->
+        <axis xyz="0 0 1" />
         <!-- <limit lower="-0.5" upper="0.5" effort="10" velocity="1" /> -->
     </joint>
